Commit message: GPS mapped to base_link (watch EKF.UAML)

File: src/ugv_main/ugv_description/urdf/ugv_rover.urdf (robot description, URDF)
Before this commit: robot ugv_rover, 13 links, 12 joints
Links:
- added link gps
Joints:
- added joint gps_joint: type fixed, parent base_link, child gps, origin xyz=0.1 0 0.2 rpy=0 0 0
